File: Circuit/boneIO - input board_BBB/boneIO_input board_BBB.kicad_pcb (KiCad board)
At the start: 2 copper layers, 256 x 74 mm, 300 parts, among them J1 ZASILACZ, J10 Conn_02x04_Odd_Even, J11 Screw_Terminal_01x04, J12 Screw_Terminal_01x08, J13 Screw_Terminal_01x08, J14 Screw_Terminal_01x08, J2 Screw_Terminal_01x08, J3 BeagleBone_Black_Header, J4 BeagleBone_Black_Header, J5 Screw_Terminal_01x08, J6 Screw_Terminal_01x08, J7 Screw_Terminal_01x08, J8 Screw_Terminal_01x08, J9 Screw_Terminal_01x08, Q1 BC817, Q2 BSS138, Q3 BC807, Q4 BC817, Q5 BC807, Q6 BSS138, SW1 SW_Push, U1 PC817X2NIP0F, U10 PC817X2NIP0F, U11 PC817X2NIP0F, U12 PC817X2NIP0F, U13 PC817X2NIP0F, U14 PC817X2NIP0F, U15 PC817X2NIP0F, U16 PC817X2NIP0F, U17 RS485, U18 PC817X2NIP0F, U19 PC817X2NIP0F, U2 LM2596S-ADJ, U20 PC817X2NIP0F, U21 PC817X2NIP0F, U22 PC817X2NIP0F, U23 PC817X2NIP0F, U24 PC817X2NIP0F, U25 PC817X2NIP0F, U26 PC817X2NIP0F, U27 PC817X2NIP0F, U28 PC817X2NIP0F, U29 PC817X2NIP0F, U3 PC817X2NIP0F, U30 PC817X2NIP0F, U31 PC817X2NIP0F, U32 P82B96, U33 PC817X2NIP0F, U34 PC817X2NIP0F, U35 PC817X2NIP0F, U36 PC817X2NIP0F, U37 PC817X2NIP0F, U38 PC817X2NIP0F, U39 PC817X2NIP0F, U4 AMS1117-3.3, U40 PC817X2NIP0F, U41 PC817X2NIP0F, U42 PC817X2NIP0F, U43 PC817X2NIP0F, U44 PC817X2NIP0F, U45 PC817X2NIP0F, U46 PC817X2NIP0F, U47 PC817X2NIP0F, U48 PC817X2NIP0F, U49 PC817X2NIP0F, U5 DS1307Z+, U50 PC817X2NIP0F, U51 PC817X2NIP0F, U52 PC817X2NIP0F, U53 PC817X2NIP0F, U54 PC817X2NIP0F, U55 PC817X2NIP0F, U56 PC817X2NIP0F, U57 PC817X2NIP0F, U58 PC817X2NIP0F, U59 PC817X2NIP0F, U6 PC817X2NIP0F, U60 PC817X2NIP0F, U61 PC817X2NIP0F, U62 PC817X2NIP0F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

Commit message: corrected version
Parts:
- J1: value ZASILACZ -> EXT_PSU
- renumbered VDD1 to VDD, ANVDD1 to VDD_ADC
Routing:
- net GND: vias 363 -> 365
Other:
- board text added: "GND_ADC"

Commit message: corrected numbering
Parts:
- renumbered VDD to J15, VDD_ADC to J16, I2C1 to J17
Other:
- board text added: "VDD"
- board text added: "VDD_ADC"
