File: Circuit/boneIO - input board_BBB/boneIO_input board_BBB.sch (KiCad schematic (older format))
At the start: 298 parts, among them J1 ZASILACZ, J10 Conn_02x04_Odd_Even, J11 Screw_Terminal_01x04, J12 Screw_Terminal_01x08, J13 Screw_Terminal_01x08, J14 Screw_Terminal_01x08, J2 Screw_Terminal_01x08, J3 BeagleBone_Black_Header, J4 BeagleBone_Black_Header, J5 Screw_Terminal_01x08, J6 Screw_Terminal_01x08, J7 Screw_Terminal_01x08, J8 Screw_Terminal_01x08, J9 Screw_Terminal_01x08, Q1 BC817, Q2 BSS138, Q3 BC807, Q4 BC817, Q5 BC807, Q6 BSS138, SW1 SW_Push, U1 PC817X2NIP0F, U10 PC817X2NIP0F, U11 PC817X2NIP0F, U12 PC817X2NIP0F, U13 PC817X2NIP0F, U14 PC817X2NIP0F, U15 PC817X2NIP0F, U16 PC817X2NIP0F, U17 RS485, U18 PC817X2NIP0F, U19 PC817X2NIP0F, U2 LM2596S-ADJ, U20 PC817X2NIP0F, U21 PC817X2NIP0F, U22 PC817X2NIP0F, U23 PC817X2NIP0F, U24 PC817X2NIP0F, U25 PC817X2NIP0F, U26 PC817X2NIP0F, U27 PC817X2NIP0F, U28 PC817X2NIP0F, U29 PC817X2NIP0F, U3 PC817X2NIP0F, U30 PC817X2NIP0F, U31 PC817X2NIP0F, U32 P82B96, U33 PC817X2NIP0F, U34 PC817X2NIP0F, U35 PC817X2NIP0F, U36 PC817X2NIP0F, U37 PC817X2NIP0F, U38 PC817X2NIP0F, U39 PC817X2NIP0F, U4 AMS1117-3.3, U40 PC817X2NIP0F, U41 PC817X2NIP0F, U42 PC817X2NIP0F, U43 PC817X2NIP0F, U44 PC817X2NIP0F, U45 PC817X2NIP0F, U46 PC817X2NIP0F, U47 PC817X2NIP0F, U48 PC817X2NIP0F, U49 PC817X2NIP0F, U5 DS1307Z+, U50 PC817X2NIP0F, U51 PC817X2NIP0F, U52 PC817X2NIP0F, U53 PC817X2NIP0F, U54 PC817X2NIP0F, U55 PC817X2NIP0F, U56 PC817X2NIP0F, U57 PC817X2NIP0F, U58 PC817X2NIP0F, U59 PC817X2NIP0F, U6 PC817X2NIP0F, U60 PC817X2NIP0F, U61 PC817X2NIP0F, U62 PC817X2NIP0F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

Commit message: corrected version
Parts:
- J1: value ZASILACZ -> EXT_PSU
Other:
- note added: "Automatic PSU Switch\n\n\n"
- note added: "BeagleBone Black"
- note added: "Clock RTC\n\n\n"
- note added: "Pin Down Relay\n\n"
- note added: "Pin Out\n\n\n\n"
- note added: "Pinout RS485 and I2C\n\n\n\n\n"
- note added: "Power Supply"
- note removed: "Automatic Power Change\n\n\n"
- note removed: "BeagleBone_Black"
- note removed: "Clock_RTC\n\n\n"
- note removed: "PINOUT_ RS485_ I2C\n\n\n\n\n"
- note removed: "PinOut\n\n\n\n"
- note removed: "Pin_Down_PCB\n\n"
- note removed: "Power"
Changed lines of the file:
@@
 	2100 5750 2250 5750
 Connection ~ 2250 5750
-Text Notes 3100 5250 0    157  ~ 31
-Power
+Text Notes 2550 5050 0    157  ~ 31
+Power Supply
 $Comp
 L Device:R R15
@@
 $EndComp
 Text Notes 27550 4150 0    157  ~ 31
-BeagleBone_Black
+BeagleBone Black
 Text GLabel 11550 9050 0    50   Input ~ 0
 P8.16_OUT
@@
 Text GLabel 17650 12100 0    50   Input ~ 0
 P9.21_OUT
-Text Notes 25900 9700 0    157  ~ 31
+Text Notes 26150 9650 0    157  ~ 31
 RS485\n\n\n\n
 Text Notes 24450 17500 0    157  ~ 31
-PinOut\n\n\n\n
+Pin Out\n\n\n\n
 Text Notes 10900 9000 0    157  ~ 31
 Transoptors\n\n\n\n
@@
 EndData
 $EndBitmap
-Text Notes 30800 9750 0    157  ~ 31
-PINOUT_ RS485_ I2C\n\n\n\n\n
+Text Notes 29000 9800 0    157  ~ 31
+Pinout RS485 and I2C\n\n\n\n\n
 Wire Notes Line
 	28550 8250 28550 11150
-Connection ~ 30850 18400
-Connection ~ 30850 18300
-Connection ~ 30850 18200
 Wire Wire Line
 	30350 18400 29700 18400
@@
 Wire Notes Line
 	32150 3650 32150 21000
-Connection ~ 31200 18400
 $Comp
 L power:GND #PWR0287
@@
 $EndComp
 Wire Wire Line
-	31200 18400 31200 18750
-Wire Wire Line
 	29700 18400 29700 17950
-Wire Wire Line
-	31200 18300 31200 18400
 Text Notes 31400 17050 2    157  ~ 31
-Pin_Down_PCB\n\n
+Pin Down Relay\n\n
 Text GLabel 30350 18500 0    50   Input ~ 0
 SCL
-Text GLabel 30850 18500 2    50   Input ~ 0
-SDA
-Connection ~ 31200 18300
-Wire Wire Line
-	30850 18300 31200 18300
-Wire Wire Line
-	31200 18200 31200 18300
-Wire Wire Line
-	30850 18200 31200 18200
-Wire Wire Line
-	30850 18400 31200 18400
-Wire Wire Line
-	30800 18400 30850 18400
 Wire Wire Line
 	29900 18300 29900 17950
 Wire Wire Line
-	30800 18300 30850 18300
-Wire Wire Line
 	30100 18200 30100 17950
-Wire Wire Line
-	30800 18200 30850 18200
 $Comp
 L power:+3.3V #PWR0265
@@
 $EndComp
 $Comp
-L Connector_Generic:Conn_02x04_Odd_Even J10
-U 1 1 61855C49
-P 30550 18300
-F 0 "J10" H 30600 18617 50  0000 C CNN
-F 1 "Conn_02x04_Odd_Even" H 30600 18526 50  0000 C CNN
-F 2 "Connector_PinSocket_2.54mm:PinSocket_2x04_P2.54mm_Vertical" H 30550 18300 50  0001 C CNN
-F 3 "~" H 30550 18300 50  0001 C CNN
-	1    30550 18300
-	1    0    0    -1
-$EndComp
-$Comp
 L Connector_Generic:Conn_02x23_Odd_Even J3
 U 1 1 64765995
@@
 P 22400 4700
 F 0 "J1" H 22480 4692 50  0000 L CNN
-F 1 "ZASILACZ" H 22480 4601 50  0000 L CNN
+F 1 "EXT_PSU" H 22480 4601 50  0000 L CNN
 F 2 "Connector_Phoenix_MSTB:PhoenixContact_MSTBA_2,5_2-G_1x02_P5.00mm_Horizontal" H 22400 4700 50  0001 C CNN
 F 3 "~" H 22400 4700 50  0001 C CNN
@@
 	21750 4600 22200 4600
 Text Notes 20250 4700 0    157  ~ 31
-Automatic Power Change\n\n\n
+Automatic PSU Switch\n\n\n
 Text Notes 15350 3550 0    394  ~ 79
 Input Board v0.3 BBB\n\n\n
@@
 $EndComp
 Text Notes 13950 4950 0    157  ~ 31
-Clock_RTC\n\n\n
+Clock RTC\n\n\n
 Wire Wire Line
 	14950 5300 14950 5600
@@
 	1    0    0    -1
 $EndComp
-Text Notes 10150 4450 0    157  ~ 31
+Text Notes 10000 4450 0    157  ~ 31
 Logic Level Converter
 $Comp
@@
 Wire Wire Line
 	26400 7550 26400 7400
+$Comp
+L Connector_Generic:Conn_02x04_Odd_Even J10
+U 1 1 61855C49
+P 30550 18300
+F 0 "J10" H 30600 18617 50  0000 C CNN
+F 1 "Conn_02x04_Odd_Even" H 30600 18526 50  0000 C CNN
+F 2 "Connector_PinSocket_2.54mm:PinSocket_2x04_P2.54mm_Vertical" H 30550 18300 50  0001 C CNN
+F 3 "~" H 30550 18300 50  0001 C CNN
+	1    30550 18300
+	1    0    0    -1
+$EndComp
+Wire Wire Line
+	30850 18400 31200 18400
+Wire Wire Line
+	30850 18200 31200 18200
+Wire Wire Line
+	31200 18200 31200 18300
+Wire Wire Line
+	30850 18300 31200 18300
+Connection ~ 31200 18300
+Text GLabel 30850 18500 2    50   Input ~ 0
+SDA
+Wire Wire Line
+	31200 18300 31200 18400
+Wire Wire Line
+	31200 18400 31200 18750
+Connection ~ 31200 18400
 $EndSCHEMATC

Commit message: corrected numbering
Parts:
- renumbered VDD1 to J15, ANVDD1 to J16, I2C1 to J17
