File: boneIO_input board_BBB.kicad_sch (KiCad schematic)
At the start: 298 parts, among them J1 Screw_Terminal_01x08, J10 Screw_Terminal_01x04, J11 BeagleBone_Black_Header, J12 BeagleBone_Black_Header, J13 Conn_02x04_Odd_Even, J14 Screw_Terminal_01x08, J2 Screw_Terminal_01x08, J3 Screw_Terminal_01x08, J4 EXT_PSU, J5 Screw_Terminal_01x08, J6 Screw_Terminal_01x08, J7 Screw_Terminal_01x08, J8 Screw_Terminal_01x08, J9 Screw_Terminal_01x08, Q1 BSS84, SW1 SW_Push, SW2 SW_DIP_x04, U1 PC817X2NIP0F, U10 PC817X2NIP0F, U11 PC817X2NIP0F, U12 PC817X2NIP0F, U13 PC817X2NIP0F, U14 PC817X2NIP0F, U15 PC817X2NIP0F, U16 PC817X2NIP0F, U17 PC817X2NIP0F, U18 RT9013-33GB, U19 PC817X2NIP0F, U2 PC817X2NIP0F, U20 PC817X2NIP0F, U21 PC817X2NIP0F, U22 PC817X2NIP0F, U23 PC817X2NIP0F, U24 PC817X2NIP0F, U25 PC817X2NIP0F, U26 PC817X2NIP0F, U27 2N7002DW/BSS138PS, U28 PC817X2NIP0F, U29 PC817X2NIP0F, U3 PC817X2NIP0F, U30 PC817X2NIP0F, U31 PC817X2NIP0F, U32 PC817X2NIP0F, U33 PC817X2NIP0F, U34 PC817X2NIP0F, U35 PC817X2NIP0F, U36 DS1307Z+, U37 PC817X2NIP0F, U38 PC817X2NIP0F, U39 PC817X2NIP0F, U4 PC817X2NIP0F, U40 PC817X2NIP0F, U41 PC817X2NIP0F, U42 PC817X2NIP0F, U43 PC817X2NIP0F, U44 PC817X2NIP0F, U45 PC817X2NIP0F, U46 PC817X2NIP0F, U47 PC817X2NIP0F, U48 PC817X2NIP0F, U49 PC817X2NIP0F, U5 PC817X2NIP0F, U50 PC817X2NIP0F, U51 PC817X2NIP0F, U52 PC817X2NIP0F, U53 PC817X2NIP0F, U54 SN65HVD230, U55 RS485, U56 P82B715DR, U57 DS2482S-100+, U58 P82B96, U59 INA226, U6 PC817X2NIP0F, U7 PC817X2NIP0F, U8 PC817X2NIP0F, U9 LM2596S-ADJ, Y1 32,788 MHz

Commit message: input board v0.5a
Parts:
- removed C11: 3n3_NC, Capacitor_SMD:C_0805_2012Metric, symbol Device:C
- removed C31, C5: 100n, Capacitor_SMD:C_0603_1608Metric, symbol Device:C
- removed JP1: 5V, Jumper:SolderJumper-2_P1.3mm_Open_Pad1.0x1.5mm, symbol Device:Jumper_NC_Small
- removed JP2: VDD_Bridge, Jumper:SolderJumper-2_P1.3mm_Bridged2Bar_RoundedPad1.0x1.5mm, symbol Jumper:Jumper_2_Bridged
- removed JP3: GND_Bridge, Jumper:SolderJumper-2_P1.3mm_Bridged2Bar_RoundedPad1.0x1.5mm, symbol Jumper:Jumper_2_Bridged
- removed JP4: VDD_Open, Jumper:SolderJumper-2_P1.3mm_Open_RoundedPad1.0x1.5mm, symbol Jumper:Jumper_2_Open
- removed JP5: GND_Open, Jumper:SolderJumper-2_P1.3mm_Open_RoundedPad1.0x1.5mm, symbol Jumper:Jumper_2_Open
- removed JP6: Jumper_NO_Small, Jumper:SolderJumper-2_P1.3mm_Open_RoundedPad1.0x1.5mm, symbol Device:Jumper_NO_Small
- removed R121: 20R_1%, Resistor_SMD:R_2512_6332Metric, symbol Device:R
- removed R17: 3k_NC, Resistor_SMD:R_0603_1608Metric, symbol Device:R
- removed U56: P82B715DR, Package_SO:SO-8_3.9x4.9mm_P1.27mm, symbol P82B715DR:P82B715DR
- removed U58: P82B96, Package_SO:SO-8_3.9x4.9mm_P1.27mm, symbol Interface_Expansion:P82B96
- removed U59: INA226, Package_SO:VSSOP-10_3x3mm_P0.5mm, symbol Analog_ADC:INA226
- removed U9: LM2596S-ADJ, Package_TO_SOT_SMD:TO-263-5_TabPin3, symbol Regulator_Switching:LM2596S-ADJ
- added C2, C29: 100n, Capacitor_SMD:C_0603_1608Metric, symbol Device:C
- added C21: 460p, Capacitor_SMD:C_0603_1608Metric, symbol Device:C
- added C?: 3.3n, Capacitor_SMD:C_0603_1608Metric, symbol Device:C
- added D12, D13, D14, D15, D16, D17, D18, D19, D2, D22, D23, D24, D25, D26, D27, D28, D29, D3, D30, D31, D32, D33, D34, D35, D36, D37, D38, D39, D4, D40, D41, D42, D43, D44, D45, D46, D47, D48, D49, D5, D50, D53, D54, D55, D56, D6, D7, D8, D9: LED, LED_SMD:LED_0603_1608Metric, symbol Device:LED_ALT
- added D62: BAT54A, Package_TO_SOT_SMD:SOT-23, symbol Diode:BAT54A
- added PWR1: Opened, Jumper:SolderJumper-2_P1.3mm_Open_RoundedPad1.0x1.5mm, symbol ESP32-EVB_Rev_I:SJ
- added R100, R101, R102, R103, R104, R105, R106, R125, R126, R127, R128, R129, R130, R131, R142, R143, R144, R145, R146, R156, R157, R158, R159, R19, R20, R21, R22, R23, R24, R25, R44, R45, R46, R47, R48, R49, R50, R51, R71, R72, R73, R74, R75, R76, R77, R78, R99: 680R, Resistor_SMD:R_0603_1608Metric, symbol Device:R
- added R171: 100R_1%, Resistor_SMD:R_2512_6332Metric, symbol Device:R
- added R9: 100k, Resistor_SMD:R_0603_1608Metric, symbol Device:R
- added R?: 1k, Resistor_SMD:R_0603_1608Metric, symbol Device:R
- added R?: 3.1k, Resistor_SMD:R_0603_1608Metric, symbol Device:R
- added U1: XL1509-5, Package_SO:SO-8_3.9x4.9mm_P1.27mm, symbol Power_Management:XL1509-5
- added U56: PCA9515, Package_SO:TSSOP-8_3x3mm_P0.65mm, symbol Interface_Expansion:PCA9515
- added U57: PCA9515, Package_SO:SO-8_3.9x4.9mm_P1.27mm, symbol Interface_Expansion:PCA9515
- added U59: INA219AxD, Package_SO:SOIC-8_3.9x4.9mm_P1.27mm, symbol Analog_ADC:INA219AxD
- C1: value 100uF/50V_NC -> 100uF/50V
- C10: renamed from C2; value 100n_NC -> 100n
- C11: renamed from C12; value 220u/35V_NC -> 100u
- C12: renamed from C18; value 100n_NC -> 100n
- C13: renamed from C14; value 100n_NC -> 100n
- C14: renamed from C15; value 100n_NC -> 100n
- C15: renamed from C16; value 100n_NC -> 100n
- C16: renamed from C17; value 100n_NC -> 100n
- C17: renamed from C19; value 100n_NC -> 100n
- C18: renamed from C20; value 100n_NC -> 100n
- C19: renamed from C21; value 100n_NC -> 100n
- C3, C4, C51, C52: value 100n_NC -> 100n
- D10: renamed from D2; value SS34_NC -> B5819W
- D11: renamed from D3; value LED_RED_NC -> LED_RED
- D61: renamed from D12; value BAT54A -> PESD5V0S2BT
- F1: value Fuse_3A -> Fuse_2A
- L2: renamed from L1; value 4.7uH_NC -> 68uH; footprint Inductor_SMD:L_12x12mm_H6mm -> Inductor_SMD:L_10.4x10.4_H4.8
- R1, R2, R3, R4, R5, R6, R7: value 4.7k -> 10k
- R107: renamed from R76; value 4.7k -> 10k
- R108: renamed from R77; value 4.7k -> 10k
- R109: renamed from R78; value 4.7k -> 10k
- R110: renamed from R79; value 4.7k -> 10k
- R111: renamed from R80; value 4.7k -> 10k
- R112: renamed from R81; value 4.7k -> 10k
- R113: renamed from R82; value 4.7k -> 10k
- R114: renamed from R83; value 4.7k -> 10k
- R124: value 10k -> 680R; JLCPCB C269704 -> C238881
- R132: renamed from R93; value 4.7k -> 10k
- R133: renamed from R94; value 4.7k -> 10k
- R134: renamed from R95; value 4.7k -> 10k
- R135: renamed from R96; value 4.7k -> 10k
- R136: renamed from R97; value 4.7k -> 10k
- R147: renamed from R103; value 4.7k -> 10k
- R148: renamed from R104; value 4.7k -> 10k
- R150: renamed from R106; value 4.7k -> 10k
- R165: renamed from R122; value 680R -> 10k
- R166: renamed from R123; value 680R -> 10k
- R18: value 1k_NC -> 680R; JLCPCB C269704 -> C238881
- R26: renamed from R27; value 330R_NC -> 330R
- R27: renamed from R23; value 4.7k -> 10k
- R28: renamed from R19; value 4.7k -> 10k
- R29: renamed from R20; value 4.7k -> 10k
- R30: renamed from R21; value 4.7k -> 10k
- R31: renamed from R22; value 4.7k -> 10k
- R32: renamed from R24; value 4.7k -> 10k
- R33: renamed from R25; value 4.7k -> 10k
- R34: renamed from R26; value 4.7k -> 10k
- R53: renamed from R38; value 4.7k -> 10k
- R54: renamed from R39; value 4.7k -> 10k
- R55: renamed from R42; value 4.7k -> 10k
- R56: renamed from R43; value 4.7k -> 10k
- R57: renamed from R44; value 4.7k -> 10k
- R58: renamed from R45; value 4.7k -> 10k
- R59: renamed from R46; value 4.7k -> 10k
- R60: renamed from R40; value 4.7k -> 10k
- R81: renamed from R58; value 4.7k -> 10k
- R82: renamed from R59; value 4.7k -> 10k
- R83: renamed from R60; value 4.7k -> 10k
- R84: renamed from R61; value 4.7k -> 10k
- R85: renamed from R62; value 4.7k -> 10k
- R86: renamed from R63; value 4.7k -> 10k
- R87: renamed from R64; value 4.7k -> 10k
- R88: renamed from R65; value 4.7k -> 10k
- U10, U11, U12, U13, U14, U15, U16, U17, U19, U20, U21, U22, U23, U24, U25, U26, U28, U29, U30, U31, U32, U33, U34, U35, U37, U38, U39, U40, U41, U42, U43, U44, U45, U46, U47, U48, U49, U50, U51, U52, U53: value PC817X2NIP0F -> EL357N; footprint PC817:SOT254P975X400-4N -> 3D_model:OPTO_EL357N-G
- U2: renamed from U1; value PC817X2NIP0F -> EL357N; footprint PC817:SOT254P975X400-4N -> 3D_model:OPTO_EL357N-G
- U3: renamed from U2; value PC817X2NIP0F -> EL357N; footprint PC817:SOT254P975X400-4N -> 3D_model:OPTO_EL357N-G
- U4: renamed from U3; value PC817X2NIP0F -> EL357N; footprint PC817:SOT254P975X400-4N -> 3D_model:OPTO_EL357N-G
- U5: renamed from U4; value PC817X2NIP0F -> EL357N; footprint PC817:SOT254P975X400-4N -> 3D_model:OPTO_EL357N-G
- U6: renamed from U5; value PC817X2NIP0F -> EL357N; footprint PC817:SOT254P975X400-4N -> 3D_model:OPTO_EL357N-G
- U7: renamed from U6; value PC817X2NIP0F -> EL357N; footprint PC817:SOT254P975X400-4N -> 3D_model:OPTO_EL357N-G
- U8: renamed from U7; value PC817X2NIP0F -> EL357N; footprint PC817:SOT254P975X400-4N -> 3D_model:OPTO_EL357N-G
- U9: renamed from U8; value PC817X2NIP0F -> EL357N; footprint PC817:SOT254P975X400-4N -> 3D_model:OPTO_EL357N-G
- renumbered C13 to C20, C24 to C23, C25 to C24, C27 to C25, C28 to C26, C29 to C27, C30 to C28, C26 to C30, C23 to C31, C6 to C5, C55 to C54, C56 to C55, C57 to C56, C58 to C57, C54 to C58, C61 to C59, C7 to C6, C59 to C60, C60 to C61, C8 to C7, C9 to C8, C10 to C9, D4 to D20, D5 to D21, D6 to D51, D7 to D52, D8 to D57, D9 to D58, D10 to D59, D11 to D60, L2 to L1, R9 to R10, R10 to R11, R84 to R115, R85 to R116, R86 to R117, R87 to R118, R88 to R119, R11 to R12, R89 to R120, R90 to R121, R91 to R122, R92 to R123, R12 to R13, R98 to R137, R99 to R138, R100 to R139, R13 to R14, R101 to R140, R102 to R141, R105 to R149, R14 to R15, R107 to R151, R108 to R152, R109 to R153, R110 to R154, R111 to R155, R15 to R16, R112 to R160, R113 to R161, R114 to R162, R115 to R163, R116 to R164, R117 to R167, R118 to R168, R119 to R169, R16 to R17, R120 to R170, R28 to R35, R29 to R36, R30 to R37, R31 to R38, R32 to R39, R33 to R40, R34 to R41, R35 to R42, R36 to R43, R37 to R52, R41 to R61, R47 to R62, R48 to R63, R49 to R64, R50 to R65, R51 to R66, R52 to R67, R53 to R68, R54 to R69, R55 to R70, R56 to R79, R57 to R80, R66 to R89, R67 to R90, R68 to R91, R69 to R92, R70 to R93, R71 to R94, R72 to R95, R73 to R96, R74 to R97, R75 to R98, U57 to U58
Connections:
- net GND_AA is gone; now on net GNDA: L4.1, L5.1, SW2.1, SW2.2
- net VDD_AA is gone; now on net VDD: L3.2, L6.2, SW2.3, SW2.4
- net +24V: now also D62.2, PWR1.2, R171.2, U1.1 (VIN), U59.7 (IN-)
- net +3V3: now also C62.2, R124.2, R18.2, R100.2, R101.2, R102.2, R103.2, R104.2, R105.2, R106.2, R125.2, R126.2, R127.2, R128.2, R129.2, R130.2, R131.2, R142.2, R143.2, R144.2, R145.2, R146.2, R156.2, R157.2, R158.2, R159.2, R19.2, R20.2, R21.2, R22.2, R23.2, R24.2, R25.2, R44.2, R45.2, R46.2, R47.2, R48.2, R49.2, R50.2, R51.2, R71.2, R72.2, R73.2, R74.2, R75.2, R76.2, R77.2, R78.2, R99.2, U56.8 (VCC), U57.8 (VCC), U59.5 (VS); no longer C62.1, R124.1, R165.1, R166.1
- net +5V: now also R165.1, R166.1, C?.2, R?.2
- net Earth: now also R9.2, R?.1, U1.5 (GND), U1.6 (GND), U1.7 (GND), U1.8 (GND); no longer R18.2
- net GND: now also C62.1, C21.2, D62.3, U56.4 (GND), U57.4 (GND), U59.1 (A1), U59.2 (A0), U59.6 (GND); no longer C12.2, C13.2, C14.2, C15.2, C16.2, C17.2, C18.2, C19.2, C23.2, C24.2, C25.2, C26.2, C27.2, C28.2, C3.2, C30.2, C32.2, C33.2, C34.2, C35.2, C36.2, C37.2, C38.2, C39.2, C4.2, C41.2, C42.2, C43.2, C44.2, C45.2, C46.2, C47.2, C48.2, C49.2, C5.2, C50.2, C51.2, C52.2, C53.2, C54.2, C55.2, C56.2, C57.2, C6.2, C62.2, C7.2, C8.2, C9.2
- net GNDA: now also C12.2, C13.2, C14.2, C15.2, C16.2, C17.2, C18.2, C19.2, C23.2, C24.2, C25.2, C26.2, C27.2, C28.2, C3.2, C30.2, C32.2, C33.2, C34.2, C35.2, C36.2, C37.2, C38.2, C39.2, C4.2, C41.2, C42.2, C43.2, C44.2, C45.2, C46.2, C47.2, C48.2, C49.2, C5.2, C50.2, C51.2, C52.2, C53.2, C54.2, C55.2, C56.2, C57.2, C6.2, C7.2, C8.2, C9.2, C2.2, C29.2
- net I2C_SCL_OUT: now also D61.2, R166.2, U56.7 (LY), U57.7 (LY); no longer D61.1, R165.2
- net I2C_SDA_OUT: now also D61.1, R165.2, U56.6 (SY), U57.6 (SY); no longer D61.2, R166.2
- net P8.07: now also D39.1 (K); no longer C42.1
- net P8.08: now also D38.1 (K); no longer C41.1
- net P8.09: now also D37.1 (K); no longer C39.1
- net P8.10: now also D36.1 (K); no longer C38.1
- net P8.11: now also D35.1 (K); no longer C37.1
- net P8.12: now also D34.1 (K); no longer C36.1
- net P8.13: now also D33.1 (K); no longer C35.1
- net P8.14: now also D32.1 (K); no longer C34.1
- net P8.15: now also D31.1 (K); no longer C33.1
- net P8.16: now also D30.1 (K); no longer C32.1
- net P8.17: now also D23.1 (K); no longer C30.1
- net P8.18: now also D22.1 (K); no longer C24.1
- net P8.19: now also D29.1 (K); no longer C23.1
- net P8.26: now also D28.1 (K)
- net P8.26_OUT: now also R59.1; no longer R59.2
- net P8.27: now also D27.1 (K); no longer C28.1
- net P8.28: now also D26.1 (K); no longer C27.1
- net P8.29: now also D25.1 (K); no longer C26.1
- net P8.30: now also D24.1 (K); no longer C25.1
- net P8.31: now also D19.1 (K); no longer C19.1
- net P8.32: now also D18.1 (K); no longer C18.1
- net P8.33: now also D17.1 (K); no longer C17.1
- net P8.33_OUT: now also R32.1; no longer R32.2
- net P8.34: now also D16.1 (K); no longer C12.1
- net P8.35: now also D15.1 (K); no longer C16.1
- net P8.36: now also D14.1 (K); no longer C15.1
- net P8.36_OUT: now also R30.1; no longer R30.2
- net P8.37: now also D13.1 (K); no longer C14.1
- net P8.38: now also D12.1 (K); no longer C13.1
- net P8.39: now also D9.1 (K); no longer C9.1
- net P8.40: now also D8.1 (K); no longer C8.1
- net P8.41: now also D7.1 (K); no longer C7.1
- net P8.42: now also D6.1 (K); no longer C6.1
- net P8.43: now also D5.1 (K); no longer C5.1
- net P8.44: now also D4.1 (K)
- net P8.45: now also D3.1 (K); no longer C4.1
- net P8.46: now also D2.1 (K); no longer C3.1
- net P9.14: now also D40.1 (K); no longer C43.1
- net P9.15: now also D41.1 (K); no longer C44.1
- net P9.16: now also D42.1 (K); no longer C45.1
- net P9.17: now also D46.1 (K); no longer C49.1
- net P9.18: now also D47.1 (K); no longer C50.1
- net P9.21: now also D48.1 (K); no longer C51.1
- net P9.22: now also D49.1 (K); no longer C52.1
- net P9.23: now also D50.1 (K); no longer C53.1
- net P9.25: now also D43.1 (K); no longer C46.1
- net P9.27: now also D44.1 (K); no longer C47.1
- net P9.28: now also D45.1 (K); no longer C48.1
- net P9.29: now also D53.1 (K); no longer C54.1
- net P9.30: now also D54.1 (K); no longer C55.1
- net P9.31: now also D55.1 (K); no longer C56.1
- net P9.42: now also D56.1 (K); no longer C57.1
- net SCL: now also U56.2 (LX), U57.2 (LX), U59.4 (SCL)
- net SDA: now also U56.3 (SX), U57.3 (SX), U59.3 (SDA)
- net VCCQ: now also D62.1, PWR1.1, R171.1, U59.8 (IN+)
- net at R2.1, U3.1: now also C3.1
- net at R18.1: now also D2.2 (A)
- net at D10.1 (K), L2.1: now also U1.2 (OUT)
- net at R3.1, U4.1: now also C4.1
- net at R4.1, U5.1: now also C5.1
- net at R5.1, U6.1: now also C6.1
- net at R6.1, U7.1: now also C7.1
- net at R7.1, U8.1: now also C8.1
- net at R8.1, U9.1: now also C9.1
- net at R28.1, U10.1: now also C13.1
- net at R29.1, U11.1: now also C14.1
- net at U12.1: now also C15.1, R30.2; no longer R30.1
- net at R31.1, U13.1: now also C16.1
- net at R27.1, U14.1: now also C12.1
- net at U15.1: now also C17.1, R32.2; no longer R32.1
- net at R33.1, U16.1: now also C18.1
- net at R34.1, U17.1: now also C19.1
- net at R55.1, U22.1: now also C25.1
- net at R56.1, U23.1: now also C26.1
- net at R57.1, U24.1: now also C27.1
- net at R58.1, U25.1: now also C28.1
- net at U26.1: now also R59.2, C29.1; no longer R59.1
- net at R110.1, U40.1: now also C44.1
- net at R111.1, U41.1: now also C45.1
- net at R83.1, U30.1: now also C34.1
- net at R82.1, U29.1: now also C33.1
- net at R81.1, U28.1: now also C32.1
- net at R54.1, U20.1: now also C24.1
- net at R60.1, U21.1: now also C30.1
- net at R107.1, U37.1: now also C41.1
- net at R88.1, U35.1: now also C39.1
- net at R87.1, U34.1: now also C38.1
- net at R86.1, U33.1: now also C37.1
- net at R85.1, U32.1: now also C36.1
- net at R114.1, U44.1: now also C48.1
- net at R113.1, U43.1: now also C47.1
- net at R53.1, U19.1: now also C23.1
- net at R112.1, U42.1: now also C46.1
- net at R109.1, U39.1: now also C43.1
- net at R147.1, U50.1: now also C54.1
- net at R133.1, U46.1: now also C50.1
- net at R134.1, U47.1: now also C51.1
- net at R135.1, U48.1: now also C52.1
- net at R84.1, U31.1: now also C35.1
- net at R136.1, U49.1: now also C53.1
- net at R132.1, U45.1: now also C49.1
- net at R1.1, U2.1: now also C2.1
- net at R108.1, U38.1: now also C42.1
- net at R150.1, U53.1: now also C57.1
- net at R149.1, U52.1: now also C56.1
- net at R148.1, U51.1: now also C55.1
- net at U18.4 (BP): now also C21.1
- new net: D53.2 (A), R156.1
- new net: D6.2 (A), R22.1
- new net: D40.2 (A), R126.1
- new net: D13.2 (A), R45.1
- new net: D16.2 (A), R48.1
- new net: D47.2 (A), R143.1
- new net: D38.2 (A), R124.1
- new net: D42.2 (A), R128.1
- new net: D9.2 (A), R25.1
- new net: D35.2 (A), R104.1
- new net: D37.2 (A), R106.1
- new net: D50.2 (A), R146.1
- new net: D55.2 (A), R158.1
- new net: D34.2 (A), R103.1
- new net: C?.1, R?.1, R?.2, U1.3 (FB)
- new net: R9.1, U1.4 (ON/OFF)
- new net: D49.2 (A), R145.1
- new net: D19.2 (A), R51.1
- new net: D18.2 (A), R50.1
- new net: D48.2 (A), R144.1
- new net: D15.2 (A), R47.1
- new net: D29.2 (A), R78.1
- new net: D56.2 (A), R159.1
- new net: D45.2 (A), R131.1
- new net: D4.2 (A), R20.1
- new net: D31.2 (A), R100.1
- new net: D43.2 (A), R129.1
- new net: D17.2 (A), R49.1
- new net: D12.2 (A), R44.1
- new net: D23.2 (A), R72.1
- new net: D22.2 (A), R71.1
- new net: D3.2 (A), R19.1
- new net: D26.2 (A), R75.1
- new net: D7.2 (A), R23.1
- new net: D44.2 (A), R130.1
- new net: D32.2 (A), R101.1
- new net: D27.2 (A), R76.1
- new net: D46.2 (A), R142.1
- new net: D41.2 (A), R127.1
- new net: D39.2 (A), R125.1
- new net: D36.2 (A), R105.1
- new net: D25.2 (A), R74.1
- new net: D33.2 (A), R102.1
- new net: D5.2 (A), R21.1
- new net: D30.2 (A), R99.1
- new net: D8.2 (A), R24.1
- new net: D54.2 (A), R157.1
- new net: D24.2 (A), R73.1
- new net: D14.2 (A), R46.1
- new net: D28.2 (A), R77.1
- no-connect marks 16 -> 15
Other:
- note added: "C22 tylko w przypadku montażu MIC5219-3.3"
- note added: "INA219"
- note removed: "INA226"
- note removed: "Transoptors"
- moved on the sheet: C11, C12, C13, C14, C15, C16, C17, C18, C19, C23, C24, C25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
