File: boneIO_input board_BBB.kicad_sch (KiCad schematic)
At the start: 299 parts, among them J1 Screw_Terminal_01x08, J10 Screw_Terminal_01x04, J11 BeagleBone_Black_Header, J12 BeagleBone_Black_Header, J13 Conn_02x04_Odd_Even, J14 Screw_Terminal_01x08, J2 Screw_Terminal_01x08, J3 Screw_Terminal_01x08, J4 EXT_PSU, J5 Screw_Terminal_01x08, J6 Screw_Terminal_01x08, J7 Screw_Terminal_01x08, J8 Screw_Terminal_01x08, J9 Screw_Terminal_01x08, Q1 BSS84, SW1 SW_Push, SW2 SW_DIP_x04, U1 PC817X2NIP0F, U10 PC817X2NIP0F, U11 PC817X2NIP0F, U12 PC817X2NIP0F, U13 PC817X2NIP0F, U14 PC817X2NIP0F, U15 PC817X2NIP0F, U16 PC817X2NIP0F, U17 PC817X2NIP0F, U18 RT9013-33GB, U19 PC817X2NIP0F, U2 PC817X2NIP0F, U20 PC817X2NIP0F, U21 PC817X2NIP0F, U22 PC817X2NIP0F, U23 PC817X2NIP0F, U24 PC817X2NIP0F, U25 PC817X2NIP0F, U26 PC817X2NIP0F, U27 2N7002DW/BSS138PS, U28 PC817X2NIP0F, U29 PC817X2NIP0F, U3 PC817X2NIP0F, U30 PC817X2NIP0F, U31 PC817X2NIP0F, U32 PC817X2NIP0F, U33 PC817X2NIP0F, U34 PC817X2NIP0F, U35 PC817X2NIP0F, U36 DS1307Z+, U37 PC817X2NIP0F, U38 PC817X2NIP0F, U39 PC817X2NIP0F, U4 PC817X2NIP0F, U40 PC817X2NIP0F, U41 PC817X2NIP0F, U42 PC817X2NIP0F, U43 PC817X2NIP0F, U44 PC817X2NIP0F, U45 PC817X2NIP0F, U46 PC817X2NIP0F, U47 PC817X2NIP0F, U48 PC817X2NIP0F, U49 PC817X2NIP0F, U5 PC817X2NIP0F, U50 PC817X2NIP0F, U51 PC817X2NIP0F, U52 PC817X2NIP0F, U53 PC817X2NIP0F, U54 SN65HVD230, U55 RS485, U56 P82B715DR, U57 DS2482S-100+, U58 P82B96, U59 INA219AxD, U6 PC817X2NIP0F, U7 PC817X2NIP0F, U8 PC817X2NIP0F, U9 LM2596S-ADJ, Y1 32,788 MHz

Commit message: input board v0.5
final version
Connections:
- net I2C_SCL_OUT: now also U56.6 (SY); no longer U56.7 (LY)
- net I2C_SDA_OUT: now also U56.7 (LY); no longer U56.2 (LX)
- net SCL: now also U56.3 (SX); no longer U56.6 (SY)
- net SDA: now also U56.2 (LX); no longer U56.3 (SX)
Changed lines of the file:
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@@
     (stroke (width 0) (type default) (color 0 0 0 0))
   )
-  (wire (pts (xy 690.88 336.55) (xy 701.04 336.55))
-    (stroke (width 0) (type default) (color 0 0 0 0))
-  )
   (wire (pts (xy 102.87 151.13) (xy 107.95 151.13))
     (stroke (width 0) (type default) (color 0 0 0 0))
@@
     (stroke (width 0) (type default) (color 0 0 0 0))
   )
+  (wire (pts (xy 690.88 321.31) (xy 699.77 321.31))
+    (stroke (width 0) (type default) (color 0 0 0 0))
+  )
   (wire (pts (xy 488.95 307.34) (xy 497.84 307.34))
     (stroke (width 0) (type default) (color 0 0 0 0))
@@
     (stroke (width 0) (type default) (color 0 0 0 0))
   )
+  (wire (pts (xy 690.88 331.47) (xy 699.77 331.47))
+    (stroke (width 0) (type default) (color 0 0 0 0))
+  )
   (wire (pts (xy 90.17 509.27) (xy 93.98 509.27))
     (stroke (width 0) (type default) (color 0 0 0 0))
@@
     (stroke (width 0) (type default) (color 0 0 0 0))
   )
-  (wire (pts (xy 690.88 321.31) (xy 704.85 321.31))
-    (stroke (width 0) (type default) (color 0 0 0 0))
-  )
   (wire (pts (xy 243.84 234.95) (xy 247.65 234.95))
     (stroke (width 0) (type default) (color 0 0 0 0))
@@
     (stroke (width 0) (type default) (color 0 0 0 0))
   )
+  (wire (pts (xy 690.88 336.55) (xy 704.85 336.55))
+    (stroke (width 0) (type default) (color 0 0 0 0))
+  )
   (wire (pts (xy 179.07 232.41) (xy 179.07 229.87))
     (stroke (width 0) (type default) (color 0 0 0 0))
@@
     (stroke (width 0) (type default) (color 0 0 0 0))
   )
-  (wire (pts (xy 690.88 331.47) (xy 701.04 331.47))
-    (stroke (width 0) (type default) (color 0 0 0 0))
-  )
   (wire (pts (xy 321.31 499.11) (xy 334.01 499.11))
     (stroke (width 0) (type default) (color 0 0 0 0))
@@
     (effects (font (size 1.27 1.27) (thickness 0.254) bold) (justify left bottom))
   )
+  (label "I2C_SCL_OUT" (at 704.85 336.55 180)
+    (effects (font (size 1.27 1.27) (thickness 0.254) bold) (justify right bottom))
+  )
   (label "VDD_AA" (at 601.98 405.13 0)
     (effects (font (size 1.27 1.27)) (justify left bottom))
@@
     (effects (font (size 1.27 1.27)) (justify left bottom))
   )
+  (label "I2C_SDA_OUT" (at 704.85 326.39 180)
+    (effects (font (size 1.27 1.27) (thickness 0.254) bold) (justify right bottom))
+  )
   (label "VDD_AA" (at 567.69 441.96 180)
     (effects (font (size 1.27 1.27)) (justify right bottom))
@@
     (effects (font (size 1.27 1.27)) (justify left bottom))
   )
-  (label "I2C_SDA_OUT" (at 704.85 321.31 180)
-    (effects (font (size 1.27 1.27) (thickness 0.254) bold) (justify right bottom))
-  )
-  (label "I2C_SCL_OUT" (at 704.85 326.39 180)
-    (effects (font (size 1.27 1.27) (thickness 0.254) bold) (justify right bottom))
-  )
   (label "I2C_SDA_OUT" (at 803.91 325.12 180)
     (effects (font (size 1.27 1.27) (thickness 0.254) bold) (justify right bottom))
@@
     )
   )
-  (global_label "SCL" (shape input) (at 701.04 336.55 0) (fields_autoplaced)
+  (global_label "SCL" (shape input) (at 699.77 331.47 0) (fields_autoplaced)
     (effects (font (size 1.27 1.27)) (justify left))
-    (property "Intersheet References" "${INTERSHEET_REFS}" (id 0) (at 706.8718 336.4706 0)
+    (property "Intersheet References" "${INTERSHEET_REFS}" (id 0) (at 705.6018 331.3906 0)
       (effects (font (size 1.27 1.27)) (justify left) hide)
     )
@@
     )
   )
-  (global_label "SDA" (shape input) (at 701.04 331.47 0) (fields_autoplaced)
+  (global_label "SDA" (shape input) (at 699.77 321.31 0) (fields_autoplaced)
     (effects (font (size 1.27 1.27)) (justify left))
-    (property "Intersheet References" "${INTERSHEET_REFS}" (id 0) (at 706.9323 331.3906 0)
+    (property "Intersheet References" "${INTERSHEET_REFS}" (id 0) (at 705.6623 321.2306 0)
       (effects (font (size 1.27 1.27)) (justify left) hide)
     )

Commit message: input board v0.5 (4 Layers)
Zmiany:
- przejście z 2 na 4 warstwy
- dodanie filtra dolnoprzepustowego na wszystkie inputy
- dodanie RS485 na PCB
- usunięcie DS2482+100
_ dodanie rezystorów 0k do rozdzielenia GND
Parts:
- removed AD1: ad0, Jumper:SolderJumper-2_P1.3mm_Bridged2Bar_RoundedPad1.0x1.5mm, symbol Jumper:Jumper_2_Bridged
- removed AD2: ad1, Jumper:SolderJumper-2_P1.3mm_Open_RoundedPad1.0x1.5mm, symbol Jumper:Jumper_2_Open
- removed C4: 100n_NC, Capacitor_SMD:C_0603_1608Metric, symbol Device:C
- removed C5, C61: 100n, Capacitor_SMD:C_0603_1608Metric, symbol Device:C
- removed D12: BAT54A, Package_TO_SOT_SMD:SOT-23, symbol Diode:BAT54A
- removed D8, D9: LED_GREEN, Capacitor_SMD:C_0805_2012Metric, symbol Device:LED
- removed JP1: 5V, Jumper:SolderJumper-2_P1.3mm_Open_Pad1.0x1.5mm, symbol Device:Jumper_NC_Small
- removed JP2: VDD_Bridge, Jumper:SolderJumper-2_P1.3mm_Bridged2Bar_RoundedPad1.0x1.5mm, symbol Jumper:Jumper_2_Bridged
- removed JP3: GND_Bridge, Jumper:SolderJumper-2_P1.3mm_Bridged2Bar_RoundedPad1.0x1.5mm, symbol Jumper:Jumper_2_Bridged
- removed JP4: VDD_Open, Jumper:SolderJumper-2_P1.3mm_Open_RoundedPad1.0x1.5mm, symbol Jumper:Jumper_2_Open
- removed JP5: GND_Open, Jumper:SolderJumper-2_P1.3mm_Open_RoundedPad1.0x1.5mm, symbol Jumper:Jumper_2_Open
- removed L2: BLM21PG221SN1D, Inductor_SMD:L_0805_2012Metric, symbol Device:L
- removed Q1: BSS84, Package_TO_SOT_SMD:SOT-23, symbol Transistor_FET:BSS84
- removed R116, R68, R70, R88, R89, R90, R91, R92, R98, R99: 10k, Resistor_SMD:R_0603_1608Metric, symbol Device:R
- removed R117: 50R, Resistor_SMD:R_0603_1608Metric, symbol Device:R
- removed R119: 4.7k, Resistor_SMD:R_0603_1608Metric, symbol Device:R
- removed R120: 0R, Resistor_SMD:R_0603_1608Metric, symbol Device:R
- removed R29, R30, R31, R32, R33, R34: 10k_NC, Resistor_SMD:R_0603_1608Metric, symbol Device:R
- removed U56: P82B715DR, Package_SO:SO-8_3.9x4.9mm_P1.27mm, symbol P82B715DR:P82B715DR
- removed U57: DS2482S-100+, Package_SO:SOP-8_3.9x4.9mm_P1.27mm, symbol DS2482S-100_:DS2482S-100+
- removed U58: P82B96, Package_SO:SO-8_3.9x4.9mm_P1.27mm, symbol Interface_Expansion:P82B96
- removed U9: LM2596S-ADJ, Package_TO_SOT_SMD:TO-263-5_TabPin3, symbol Regulator_Switching:LM2596S-ADJ
- removed WIRE1: SPU, Jumper:SolderJumper-2_P1.3mm_Open_RoundedPad1.0x1.5mm, symbol Jumper:Jumper_2_Open
- added C1, C104, C105, C106, C107, C111, C12, C13, C14, C15, C16, C17, C18, C2, C29, C30, C31, C33, C34, C35, C36, C45, C48, C49, C50, C51, C52, C53, C54, C55, C64, C65, C66, C67, C68, C69, C70, C71, C81, C82, C83, C84, C85, C86, C87, C88, C94, C95, C96, C97, C98: 100n, Capacitor_SMD:C_0603_1608Metric, symbol Device:C
- added D13: PSM712, Package_TO_SOT_SMD:SOT-23, symbol Diode:BAT54A
- added D8, D9: LED_RED, LED_SMD:LED_0805_2012Metric, symbol Device:LED_ALT
- added L10, L11, L6, L7, L8, L9: BLM21, Inductor_SMD:L_0805_2012Metric, symbol Device:L_Small
- added Q1: BSS138, Package_TO_SOT_SMD:SOT-23, symbol Transistor_FET:BSS138
- added Q2: BC817, Package_TO_SOT_SMD:SOT-23, symbol Transistor_BJT:BC817
- added R103, R104, R105, R106, R107, R125, R126, R127, R128, R129, R130, R131, R132, R146, R147, R148, R149, R150, R161, R162, R163, R164, R176, R180, R40, R41, R42, R43, R44, R45, R46, R47, R76, R77, R78, R79: 10k, Resistor_SMD:R_0603_1608Metric, symbol Device:R
- added R112, R113, R114, R133, R134, R135, R136, R137, R138, R139, R140, R151, R152, R153, R154, R155, R165, R166, R167, R168, R19, R20, R21, R22, R23, R24, R25, R56, R80, R81, R82, R83, R84: 1k, Resistor_SMD:R_0603_1608Metric, symbol Device:R
- added R174, R177, R183, R184: 4.7k, Resistor_SMD:R_0603_1608Metric, symbol Device:R
- added R185, R187: 10R, Resistor_SMD:R_0603_1608Metric, symbol Device:R
- added R188: 120R, Resistor_SMD:R_0603_1608Metric, symbol Device:R
- added R37, R38, R57, R59: 0k, Resistor_SMD:R_0805_2012Metric, symbol Device:R
- added U1: HLK-5D2405, 3D_model:HLK5D2405, symbol Power_Management:HLK-5D2405
- added U2: XL1509-5, Package_SO:SO-8_3.9x4.9mm_P1.27mm, symbol Power_Management:XL1509-5
- added U57: PCA9515, Package_SO:TSSOP-8_3x3mm_P0.65mm, symbol Interface_Expansion:PCA9515
- added U59: SP3485EN, Package_SO:SOIC-8_3.9x4.9mm_P1.27mm, symbol Interface_UART:SP3485EN
- C10: renamed from C2; value 100n_NC -> 100n
- C11: value 3n3_NC -> 100n; footprint Capacitor_SMD:C_0805_2012Metric -> Capacitor_SMD:C_0603_1608Metric; JLCPCB C107149 -> C14663
- C19: renamed from C12; value 220u/35V_NC -> 100u
- C20: renamed from C18; value 100n_NC -> 100n
- C21: renamed from C14; value 100n_NC -> 100n
- C22: renamed from C15; value 100n_NC -> 100n
- C23: renamed from C16; value 100n_NC -> 100n
- C24: renamed from C17; value 100n_NC -> 100n
- C25: renamed from C19; value 100n_NC -> 100n
- C26: renamed from C20; value 100n_NC -> 100n
- C27: renamed from C21; value 100n_NC -> 100n
- C3: value 100n_NC -> 100n
- C9: renamed from C1; value 100uF/50V_NC -> 100uF/50V
- C91: renamed from C52; value 100n_NC -> 100n
- C92: renamed from C53; value 100n_NC -> 100n
- D12: renamed from D13; value BAT54A -> PESD5V0S2BT
- D2: value SS34_NC -> B5819W
- D3: value LED_RED_NC -> LED_RED
- F1: value Fuse_3A -> Fuse_2A
- L1: value 4.7uH_NC -> 68uH; footprint Inductor_SMD:L_12x12mm_H6mm -> Inductor_SMD:L_Bourns-SRN8040_8x8.15mm
- R1, R2, R3, R4, R5, R6, R7: value 4.7k -> 10k
- R10, R100, R101: value 10k_NC -> 10k; JLCPCB C238881 -> C237118
- R102, R11, R12, R13, R14, R15, R16, R72, R73, R74, R75: JLCPCB C238881 -> C237118
- R108, R109, R110, R111, R49, R50, R51, R52, R53, R54, R55, R85, R86, R87: value 10k -> 1k
- R115: value 10k -> 1k; JLCPCB (none) -> C238881
- R116: renamed from R76; value 4.7k -> 10k
- R117: renamed from R77; value 4.7k -> 10k
- R118: renamed from R78; value 4.7k -> 10k
- R119: renamed from R79; value 4.7k -> 10k
- R120: renamed from R80; value 4.7k -> 10k
- R121: renamed from R81; value 4.7k -> 10k
- R122: renamed from R82; value 4.7k -> 10k
- R141: renamed from R93; value 4.7k -> 10k
- R142: renamed from R94; value 4.7k -> 10k
- R143: renamed from R95; value 4.7k -> 10k
- R144: renamed from R96; value 4.7k -> 10k
- R145: renamed from R97; value 4.7k -> 10k
- R156: renamed from R103; value 4.7k -> 10k
- R157: renamed from R104; value 4.7k -> 10k
- R159: renamed from R106; value 4.7k -> 10k
- R17: value 3k_NC -> 10k; JLCPCB C126358 -> C237118
- R170: renamed from R113; value 330R -> 1k
- R171: renamed from R114; value 330R -> 1k
- R175: renamed from R121; value 680R -> 10k
- R178: renamed from R123; value 680R -> 10k
- R18: value 1k_NC -> 1k; JLCPCB C269704 -> C238881
- R26: renamed from R27; value 330R_NC -> 1k
- R27: renamed from R23; value 4.7k -> 10k
- R28: renamed from R19; value 4.7k -> 10k
- R29: renamed from R20; value 4.7k -> 10k
- R30: renamed from R21; value 4.7k -> 10k
- R31: renamed from R22; value 4.7k -> 10k
- R32: renamed from R24; value 4.7k -> 10k
- R33: renamed from R25; value 4.7k -> 10k
- R34: renamed from R26; value 4.7k -> 10k
- R35, R36: value 10k_NC -> 0k; footprint Resistor_SMD:R_0603_1608Metric -> Resistor_SMD:R_0805_2012Metric; JLCPCB C238881 -> (none)
- R48, R69, R71: value 10k -> 0k; footprint Resistor_SMD:R_0603_1608Metric -> Resistor_SMD:R_0805_2012Metric; JLCPCB C238881 -> (none)
- R58: renamed from R37; value 330R -> 1k
- R60: renamed from R38; value 4.7k -> 10k
- R61: renamed from R39; value 4.7k -> 10k
- R62: renamed from R42; value 4.7k -> 10k
- R63: renamed from R43; value 4.7k -> 10k
- R64: renamed from R44; value 4.7k -> 10k
- R65: renamed from R45; value 4.7k -> 10k
- R66: renamed from R46; value 4.7k -> 10k
- R67: renamed from R40; value 4.7k -> 10k
- R9: value 10k_NC -> 100k; JLCPCB C238881 -> C269704
- R90: renamed from R58; value 4.7k -> 10k
- R91: renamed from R59; value 4.7k -> 10k
- R92: renamed from R60; value 4.7k -> 10k
- R93: renamed from R61; value 4.7k -> 10k
- R94: renamed from R62; value 4.7k -> 10k
- R95: renamed from R63; value 4.7k -> 10k
- R96: renamed from R64; value 4.7k -> 10k
- R97: renamed from R65; value 4.7k -> 10k
- U10: renamed from U8; value PC817X2NIP0F -> EL357N; footprint PC817:SOT254P975X400-4N -> 3D_model:OPTO_EL357N-G
- U11: renamed from U10; value PC817X2NIP0F -> EL357N; footprint PC817:SOT254P975X400-4N -> 3D_model:OPTO_EL357N-G
- U12: renamed from U11; value PC817X2NIP0F -> EL357N; footprint PC817:SOT254P975X400-4N -> 3D_model:OPTO_EL357N-G
- U13: renamed from U12; value PC817X2NIP0F -> EL357N; footprint PC817:SOT254P975X400-4N -> 3D_model:OPTO_EL357N-G
- U14: renamed from U13; value PC817X2NIP0F -> EL357N; footprint PC817:SOT254P975X400-4N -> 3D_model:OPTO_EL357N-G
- U15: renamed from U14; value PC817X2NIP0F -> EL357N; footprint PC817:SOT254P975X400-4N -> 3D_model:OPTO_EL357N-G
- U16: renamed from U15; value PC817X2NIP0F -> EL357N; footprint PC817:SOT254P975X400-4N -> 3D_model:OPTO_EL357N-G
- U17: renamed from U16; value PC817X2NIP0F -> EL357N; footprint PC817:SOT254P975X400-4N -> 3D_model:OPTO_EL357N-G
- U18: renamed from U17; value PC817X2NIP0F -> EL357N; footprint PC817:SOT254P975X400-4N -> 3D_model:OPTO_EL357N-G
- U20: renamed from U19; value PC817X2NIP0F -> EL357N; footprint PC817:SOT254P975X400-4N -> 3D_model:OPTO_EL357N-G
- U21: renamed from U20; value PC817X2NIP0F -> EL357N; footprint PC817:SOT254P975X400-4N -> 3D_model:OPTO_EL357N-G
- U22: renamed from U21; value PC817X2NIP0F -> EL357N; footprint PC817:SOT254P975X400-4N -> 3D_model:OPTO_EL357N-G
- U23: renamed from U22; value PC817X2NIP0F -> EL357N; footprint PC817:SOT254P975X400-4N -> 3D_model:OPTO_EL357N-G
- U24: renamed from U23; value PC817X2NIP0F -> EL357N; footprint PC817:SOT254P975X400-4N -> 3D_model:OPTO_EL357N-G
- U25: renamed from U24; value PC817X2NIP0F -> EL357N; footprint PC817:SOT254P975X400-4N -> 3D_model:OPTO_EL357N-G
- U26: renamed from U25; value PC817X2NIP0F -> EL357N; footprint PC817:SOT254P975X400-4N -> 3D_model:OPTO_EL357N-G
- U27: renamed from U26; value PC817X2NIP0F -> EL357N; footprint PC817:SOT254P975X400-4N -> 3D_model:OPTO_EL357N-G
- U29: renamed from U28; value PC817X2NIP0F -> EL357N; footprint PC817:SOT254P975X400-4N -> 3D_model:OPTO_EL357N-G
- U3: renamed from U1; value PC817X2NIP0F -> EL357N; footprint PC817:SOT254P975X400-4N -> 3D_model:OPTO_EL357N-G
- U30: renamed from U29; value PC817X2NIP0F -> EL357N; footprint PC817:SOT254P975X400-4N -> 3D_model:OPTO_EL357N-G
- U31: renamed from U30; value PC817X2NIP0F -> EL357N; footprint PC817:SOT254P975X400-4N -> 3D_model:OPTO_EL357N-G
- U32: renamed from U31; value PC817X2NIP0F -> EL357N; footprint PC817:SOT254P975X400-4N -> 3D_model:OPTO_EL357N-G
- U33: renamed from U32; value PC817X2NIP0F -> EL357N; footprint PC817:SOT254P975X400-4N -> 3D_model:OPTO_EL357N-G
- U34: renamed from U33; value PC817X2NIP0F -> EL357N; footprint PC817:SOT254P975X400-4N -> 3D_model:OPTO_EL357N-G
- U35: renamed from U34; value PC817X2NIP0F -> EL357N; footprint PC817:SOT254P975X400-4N -> 3D_model:OPTO_EL357N-G
- U36: renamed from U35; value PC817X2NIP0F -> EL357N; footprint PC817:SOT254P975X400-4N -> 3D_model:OPTO_EL357N-G
- U38: renamed from U37; value PC817X2NIP0F -> EL357N; footprint PC817:SOT254P975X400-4N -> 3D_model:OPTO_EL357N-G
- U39: renamed from U38; value PC817X2NIP0F -> EL357N; footprint PC817:SOT254P975X400-4N -> 3D_model:OPTO_EL357N-G
- U4: renamed from U2; value PC817X2NIP0F -> EL357N; footprint PC817:SOT254P975X400-4N -> 3D_model:OPTO_EL357N-G
- U40: renamed from U39; value PC817X2NIP0F -> EL357N; footprint PC817:SOT254P975X400-4N -> 3D_model:OPTO_EL357N-G
- U41: renamed from U40; value PC817X2NIP0F -> EL357N; footprint PC817:SOT254P975X400-4N -> 3D_model:OPTO_EL357N-G
- U42: renamed from U41; value PC817X2NIP0F -> EL357N; footprint PC817:SOT254P975X400-4N -> 3D_model:OPTO_EL357N-G
- U43: renamed from U42; value PC817X2NIP0F -> EL357N; footprint PC817:SOT254P975X400-4N -> 3D_model:OPTO_EL357N-G
- U44: renamed from U43; value PC817X2NIP0F -> EL357N; footprint PC817:SOT254P975X400-4N -> 3D_model:OPTO_EL357N-G
- U45: renamed from U44; value PC817X2NIP0F -> EL357N; footprint PC817:SOT254P975X400-4N -> 3D_model:OPTO_EL357N-G
- U46: renamed from U45; value PC817X2NIP0F -> EL357N; footprint PC817:SOT254P975X400-4N -> 3D_model:OPTO_EL357N-G
- U47: renamed from U46; value PC817X2NIP0F -> EL357N; footprint PC817:SOT254P975X400-4N -> 3D_model:OPTO_EL357N-G
- U48: renamed from U47; value PC817X2NIP0F -> EL357N; footprint PC817:SOT254P975X400-4N -> 3D_model:OPTO_EL357N-G
- U49: renamed from U48; value PC817X2NIP0F -> EL357N; footprint PC817:SOT254P975X400-4N -> 3D_model:OPTO_EL357N-G
- U5: renamed from U3; value PC817X2NIP0F -> EL357N; footprint PC817:SOT254P975X400-4N -> 3D_model:OPTO_EL357N-G
- U50: renamed from U49; value PC817X2NIP0F -> EL357N; footprint PC817:SOT254P975X400-4N -> 3D_model:OPTO_EL357N-G
- U51: renamed from U50; value PC817X2NIP0F -> EL357N; footprint PC817:SOT254P975X400-4N -> 3D_model:OPTO_EL357N-G
- U52: renamed from U51; value PC817X2NIP0F -> EL357N; footprint PC817:SOT254P975X400-4N -> 3D_model:OPTO_EL357N-G
- U53: renamed from U52; value PC817X2NIP0F -> EL357N; footprint PC817:SOT254P975X400-4N -> 3D_model:OPTO_EL357N-G
- U54: renamed from U53; value PC817X2NIP0F -> EL357N; footprint PC817:SOT254P975X400-4N -> 3D_model:OPTO_EL357N-G
- U6: renamed from U4; value PC817X2NIP0F -> EL357N; footprint PC817:SOT254P975X400-4N -> 3D_model:OPTO_EL357N-G
- U7: renamed from U5; value PC817X2NIP0F -> EL357N; footprint PC817:SOT254P975X400-4N -> 3D_model:OPTO_EL357N-G
- U8: renamed from U6; value PC817X2NIP0F -> EL357N; footprint PC817:SOT254P975X400-4N -> 3D_model:OPTO_EL357N-G
- U9: renamed from U7; value PC817X2NIP0F -> EL357N; footprint PC817:SOT254P975X400-4N -> 3D_model:OPTO_EL357N-G
- renumbered C57 to C100, C58 to C101, C59 to C102, C55 to C103, C62 to C108, C60 to C109, C63 to C112, C13 to C28, C22 to C37, C23 to C38, C25 to C39, C6 to C4, C26 to C40, C28 to C41, C29 to C42, C30 to C43, C31 to C44, C27 to C46, C24 to C47, C7 to C5, C33 to C56, C34 to C57, C35 to C58, C36 to C59, C8 to C6, C37 to C60, C38 to C61, C39 to C62, C40 to C63, C9 to C7, C41 to C72, C42 to C73, C43 to C74, C44 to C75, C45 to C76, C46 to C77, C47 to C78, C48 to C79, C10 to C8, C49 to C80, C50 to C89, C51 to C90, C54 to C93, C56 to C99, L3 to L2, L4 to L3, L5 to L4, L6 to L5, R83 to R123, R84 to R124, R105 to R158, R107 to R160, R112 to R169, R118 to R182, R122 to R186, R28 to R39, R41 to R68, R47 to R70, R56 to R88, R57 to R89, R66 to R98, R67 to R99, U18 to U19, U27 to U28, U36 to U37, U54 to U55, U55 to U56, U59 to U60
Connections:
- net +24V: now also U1.2 (+Vin), U2.1 (VIN)
- net +3V3: now also D8.2 (A), D9.2 (A), L10.1, Q1.1 (G), R174.2, U57.8 (VCC); no longer J13.5 (Pin_5), R10.2, R100.2, R101.2, R102.2, R108.2, R109.2, R11.2, R110.2, R111.2, R12.2, R13.2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
- net +5V: now also R175.1, R178.1, R177.2, U1.3 (VO+), U2.3 (FB); no longer C11.1, R17.1
- net 1-Wire: now also Q1.3 (D), R177.1
- net 1-Wire_OUT: now also Q1.2 (S), R174.1
- net A+_OUT: now also D13.2, R183.1, R188.2, U59.6 (A)
- net B-_OUT: now also D13.1, R184.2, R188.1, U59.7 (B)
- net Earth: now also J13.2 (Pin_2), J13.4 (Pin_4), L3.2, R48.2, R69.2, R71.2, SW2.4, R38.2, R57.2, R59.2; no longer C10.2, C19.2, C9.2, D2.2 (A), D3.1 (K), R18.2
- net GND: now also R36.1, R48.1, L11.2, R37.1, R38.1, U1.5 (GND), U57.4 (GND); no longer C100.2, C101.2, C102.2, C112.1, C20.2, C21.2, C22.2, C23.2, C24.2, C25.2, C26.2, C27.2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
- net GND1: now also SW2.3; no longer SW2.7
- net GNDA: now also C100.2, C101.2, C102.2, C20.2, C21.2, C22.2, C23.2, C24.2, C25.2, C26.2, C27.2, C3.2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
- net GND_AA: now also SW2.5, SW2.6, L7.1, L8.1; no longer SW2.1, SW2.2
- net I2C_SCL_OUT: now also D12.2, R178.2, U57.7 (LY); no longer D12.1, R175.2
- net I2C_SDA_OUT: now also D12.1, R175.2, U57.6 (SY); no longer D12.2, R178.2
- net P8.07: now also C82.1, R134.2; no longer C74.1, R86.1, U39.4
- net P8.08: now also C81.1, R133.2; no longer C73.1, R85.1, U38.4
- net P8.09: now also R115.2, C71.1; no longer C63.1, R75.1, U36.4
- net P8.10: now also C70.1, R114.2; no longer C62.1, R74.1, U35.4
- net P8.11: now also C69.1, R113.2; no longer C61.1, R73.1, U34.4
- net P8.12: now also C68.1, R112.2; no longer C60.1, R72.1, U33.4
- net P8.13: now also R111.2, C67.1; no longer C59.1, R71.1, U32.4
- net P8.14: now also R110.2, C66.1; no longer C58.1, U31.4
- net P8.15: now also R109.2, C65.1; no longer C57.1, R69.1, U30.4
- net P8.16: now also R108.2, C64.1; no longer C56.1, U29.4
- net P8.17: now also C50.1, R82.2; no longer C46.1, R50.1, U22.4
- net P8.18: now also C49.1, R81.2; no longer C40.1, R49.1, U21.4
- net P8.19: now also C48.1, R80.2; no longer C39.1, R48.1, U20.4
- net P8.26: now also R87.2, C55.1; no longer C32.1, R55.1, U27.4
- net P8.26_OUT: now also R66.1; no longer R66.2
- net P8.27: now also R86.2, C54.1; no longer C44.1, R54.1, U26.4
- net P8.28: now also R85.2, C53.1; no longer C43.1, R53.1, U25.4
- net P8.29: now also C52.1, R84.2; no longer C42.1, R52.1, U24.4
- net P8.30: now also C51.1, R83.2; no longer C41.1, R51.1, U23.4
- net P8.31: now also C36.1, R56.2; no longer C27.1, R36.1, U18.4
- net P8.32: now also R55.2, C35.1; no longer C26.1, R35.1, U17.4
- net P8.33: now also R54.2, C34.1; no longer C25.1, U16.4
- net P8.33_OUT: now also R32.1; no longer R32.2
- net P8.34: now also R53.2, C33.1; no longer C20.1, U15.4
- net P8.35: now also C32.1, R52.2; no longer C24.1, U14.4
- net P8.36: now also R51.2, C31.1; no longer C23.1, U13.4
- net P8.36_OUT: now also R30.1; no longer R30.2
- net P8.37: now also R50.2, C30.1; no longer C22.1, U12.4
- net P8.38: now also R49.2, C29.1; no longer C21.1, U11.4
- net P8.39: now also C18.1, R25.2; no longer C8.1, R16.1, U10.4
- net P8.40: now also C17.1, R24.2; no longer C7.1, R15.1, U9.4
- net P8.41: now also C16.1, R23.2; no longer C6.1, R14.1, U8.4
- net P8.42: now also C15.1, R22.2; no longer C5.1, R13.1, U7.4
- net P8.43: now also C14.1, R21.2; no longer C4.1, R12.1, U6.4
- net P8.44: now also C13.1, R20.2; no longer R11.1, U5.4
- net P8.45: now also C12.1, R19.2; no longer R10.1, U4.4
- net P8.46: now also C11.1, R18.2; no longer C3.1, R9.1, U3.4
- net P9.14: now also C83.1, R135.2; no longer C75.1, R87.1, U40.4
- net P9.15: now also C84.1, R136.2; no longer C76.1, U41.4
- net P9.16: now also C85.1, R137.2; no longer C77.1, U42.4
- net P9.17: now also C94.1, R151.2; no longer C89.1, U46.4
- net P9.18: now also C95.1, R152.2; no longer C90.1, U47.4
- net P9.21: now also C96.1, R153.2; no longer C91.1, R100.1, U48.4
- net P9.22: now also C97.1, R154.2; no longer C92.1, R101.1, U49.4
- net P9.23: now also C98.1, R155.2; no longer C93.1, R102.1, U50.4
- net P9.25: now also C86.1, R138.2; no longer C78.1, U43.4
- net P9.27: now also C87.1, R139.2; no longer C79.1, U44.4
- net P9.28: now also C88.1, R140.2; no longer C80.1, U45.4
- net P9.29: now also C104.1, R165.2; no longer C99.1, R108.1, U51.4
- net P9.30: now also C105.1, R166.2; no longer C100.1, R109.1, U52.4
- net P9.31: now also C106.1, R167.2; no longer C101.1, R110.1, U53.4
- net P9.42: now also C107.1, R168.2; no longer C102.1, R111.1, U54.4
- net RS485_RX: now also U59.1 (RO)
- net RS485_TX: now also R176.1, U59.4 (DI)
- net SCL: now also R185.1, U57.2 (LX); no longer J13.7 (Pin_7)
- new net: R11.1, R19.1, U4.4
- new net: J13.7 (Pin_7), R185.2
- new net: J13.8 (Pin_8), R187.2
- new net: R12.1, R20.1, U5.4
- new net: R13.1, R21.1, U6.4
- new net: R14.1, R22.1, U7.4
- new net: R15.1, R23.1, U8.4
- new net: R16.1, R24.1, U9.4
- new net: R17.1, R25.1, U10.4
- new net: R40.1, R49.1, U11.4
- new net: R41.1, R50.1, U12.4
- new net: R42.1, R51.1, U13.4
- new net: R43.1, R52.1, U14.4
- new net: R44.1, R53.1, U15.4
- new net: R45.1, R54.1, U16.4
- new net: R46.1, R55.1, U17.4
- new net: R47.1, R56.1, U18.4
- new net: R75.1, R83.1, U23.4
- new net: R76.1, R84.1, U24.4
- new net: R77.1, R85.1, U25.4
- new net: R78.1, R86.1, U26.4
- new net: R79.1, R87.1, U27.4
- new net: R128.1, R136.1, U41.4
- new net: R129.1, R137.1, U42.4
- new net: R102.1, R110.1, U31.4
- new net: R101.1, R109.1, U30.4
- new net: R100.1, R108.1, U29.4
- new net: R73.1, R81.1, U21.4
- new net: R74.1, R82.1, U22.4
- new net: R125.1, R133.1, U38.4
- new net: R106.1, R114.1, U35.4
- new net: R105.1, R113.1, U34.4
- new net: R104.1, R112.1, U33.4
- new net: R132.1, R140.1, U45.4
- new net: R131.1, R139.1, U44.4
- new net: R72.1, R80.1, U20.4
- new net: R130.1, R138.1, U43.4
- new net: R127.1, R135.1, U40.4
- new net: R161.1, R165.1, U51.4
- new net: R147.1, R152.1, U47.4
- new net: R148.1, R153.1, U48.4
- new net: R149.1, R154.1, U49.4
- new net: R103.1, R111.1, U32.4
- new net: R150.1, R155.1, U50.4
- new net: R146.1, R151.1, U46.4
- new net: R10.1, R18.1, U3.4
- new net: R126.1, R134.1, U39.4
- new net: R164.1, R168.1, U54.4
- new net: R163.1, R167.1, U53.4
- new net: R162.1, R166.1, U52.4
- new net: R9.1, U2.4 (ON/OFF)
- new net: Q2.3 (C), R180.1, U59.2 (~{RE}), U59.3 (DE)
- new net: Q2.1 (B), R176.2
- new net +3.3VA: J13.5 (Pin_5), R10.2, R100.2, R101.2, R102.2, R103.2, R104.2, R105.2, R106.2, R107.2, R11.2, R12.2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
- new net +3.3VP: C111.2, L10.2, R180.2, R183.2, U59.8 (VCC)
- new net GND3: C104.2, C105.2, C106.2, C107.2, C11.2, C12.2, C13.2, C14.2, C15.2, C16.2, C17.2, C18.2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
- new net GNDPWR: C10.2, C112.1, C19.2, C9.2, D2.2 (A), D3.1 (K), R69.1, R71.1, R9.2, U1.1 (-Vin), U2.5 (GND), U2.6 (GND)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
- new net GNDS: C111.1, D13.3, L11.1, Q2.2 (E), R184.1, U59.5 (GND)
- new net GND_C: R57.1
- new net GND_GPIO: R59.1
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Other:
- note removed: "Transoptors"
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
Commit message: input board v0.5 with 4 layers
Parts:
- removed C104, C105, C106, C107, C11, C111, C12, C13, C14, C15, C16, C17, C18, C29, C30, C31, C32, C33, C34, C35, C36, C48, C49, C50, C51, C52, C53, C54, C55, C64, C65, C66, C67, C68, C69, C70, C71, C81, C82, C83, C84, C85, C86, C87, C88, C94, C95, C96, C97, C98: 100n, Capacitor_SMD:C_0603_1608Metric, symbol Device:C
- removed D13: PSM712, Package_TO_SOT_SMD:SOT-23, symbol Diode:BAT54A
- removed L10, L11: BLM21, Inductor_SMD:L_0805_2012Metric, symbol Device:L_Small
- removed Q1: BSS138, Package_TO_SOT_SMD:SOT-23, symbol Transistor_FET:BSS138
- removed Q2: BC817, Package_TO_SOT_SMD:SOT-23, symbol Transistor_BJT:BC817
- removed R107, R132, R147, R148, R149, R150, R161, R162, R176, R180, R79: 10k, Resistor_SMD:R_0603_1608Metric, symbol Device:R
- removed R108, R109, R110, R111, R112, R113, R114, R115, R133, R134, R135, R136, R151, R165, R166, R168, R52, R53, R54, R55, R56, R80, R81, R82, R83, R84, R85, R86, R87: 1k, Resistor_SMD:R_0603_1608Metric, symbol Device:R
- removed R174, R177, R183, R184: 4.7k, Resistor_SMD:R_0603_1608Metric, symbol Device:R
- removed R185, R187: 10R, Resistor_SMD:R_0603_1608Metric, symbol Device:R
- removed R188: 120R, Resistor_SMD:R_0603_1608Metric, symbol Device:R
- removed R35, R57, R59: 0k, Resistor_SMD:R_0805_2012Metric, symbol Device:R
- removed U59: SP3485EN, Package_SO:SOIC-8_3.9x4.9mm_P1.27mm, symbol Interface_UART:SP3485EN
- added AD1: ad0, Jumper:SolderJumper-2_P1.3mm_Bridged2Bar_RoundedPad1.0x1.5mm, symbol Jumper:Jumper_2_Bridged
- added AD2: ad1, Jumper:SolderJumper-2_P1.3mm_Open_RoundedPad1.0x1.5mm, symbol Jumper:Jumper_2_Open
- added C61: 100n, Capacitor_SMD:C_0603_1608Metric, symbol Device:C
- added D12, D13, D14, D15, D16, D17, D18, D19, D2, D22, D23, D24, D25, D26, D27, D28, D29, D3, D30, D31, D32, D33, D34, D35, D36, D37, D38, D39, D4, D40, D41, D42, D43, D44, D45, D46, D47, D48, D49, D5, D50, D53, D54, D55, D56, D6, D7: LED, LED_SMD:LED_0603_1608Metric, symbol Device:LED_ALT
- added D57, D58: LED_GREEN, Capacitor_SMD:C_0805_2012Metric, symbol Device:LED
- added L2, L3: BLM21, Inductor_SMD:L_0805_2012Metric, symbol Device:L_Small
- added Q1: BSS84, Package_TO_SOT_SMD:SOT-23, symbol Transistor_FET:BSS84
- added R116, R117, R118, R119, R120, R121, R122, R141, R63, R64, R65, R66, R67, R68, R70, R91, R92, R93, R94, R95, R96, R97, R98: 10k, Resistor_SMD:R_0603_1608Metric, symbol Device:R
- added R123: 1.5k, Resistor_SMD:R_0603_1608Metric, symbol Device:R
- added R124, R142, R143, R144, R145, R156, R157, R158, R159, R99: 680R, Resistor_SMD:R_0603_1608Metric, symbol Device:R
- added R169: 4.7k, Resistor_SMD:R_0603_1608Metric, symbol Device:R
- added R170: 0R, Resistor_SMD:R_0603_1608Metric, symbol Device:R
- added R39: 10k_NC, Resistor_SMD:R_0603_1608Metric, symbol Device:R
- added U58: PCA9515, Package_SO:SO-8_3.9x4.9mm_P1.27mm, symbol Interface_Expansion:PCA9515
- added U59: DS2482S-100+, Package_SO:SOP-8_3.9x4.9mm_P1.27mm, symbol DS2482S-100_:DS2482S-100+
- added WIRE1: SPU, Jumper:SolderJumper-2_P1.3mm_Open_RoundedPad1.0x1.5mm, symbol Jumper:Jumper_2_Open
- D8, D9: value LED_RED -> LED; footprint LED_SMD:LED_0805_2012Metric -> LED_SMD:LED_0603_1608Metric
- R10, R11, R40, R41, R42, R43: value 10k -> 10k_NC; JLCPCB C237118 -> C238881
- R100, R101, R102, R103, R104, R105, R106, R125, R126, R127, R128, R129, R130, R131, R146, R44, R45, R46, R47, R72, R73, R74, R75, R76, R77, R78: value 10k -> 680R; JLCPCB C237118 -> C238881
- R12, R13, R14, R15, R16, R17: JLCPCB C237118 -> C238881
- R137, R138, R152, R153, R154, R155: value 1k -> 10k
- R139, R140: value 1k -> 10k_NC
- R161: renamed from R170; value 1k -> 330R
- R162: renamed from R171; value 1k -> 330R
- R163, R164: JLCPCB C237118 -> (none)
- R167: value 1k -> 50R; JLCPCB C238881 -> (none)
- R18, R19, R20, R21, R22, R23, R24, R25, R49, R50, R51: value 1k -> 680R
- R26: value 1k -> 330R
- R36, R37, R38: value 0k -> 10k_NC; footprint Resistor_SMD:R_0805_2012Metric -> Resistor_SMD:R_0603_1608Metric; JLCPCB (none) -> C238881
- R48, R71: value 0k -> 680R; footprint Resistor_SMD:R_0805_2012Metric -> Resistor_SMD:R_0603_1608Metric; JLCPCB (none) -> C238881
- R52: renamed from R58; value 1k -> 330R
- R69: value 0k -> 10k; footprint Resistor_SMD:R_0805_2012Metric -> Resistor_SMD:R_0603_1608Metric; JLCPCB (none) -> C238881
- renumbered C9 to C1, C19 to C11, C20 to C12, C21 to C13, C22 to C14, C23 to C15, C24 to C16, C25 to C17, C26 to C18, C27 to C19, C1 to C2, C28 to C20, C37 to C21, C38 to C22, C39 to C23, C40 to C24, C41 to C25, C42 to C26, C43 to C27, C44 to C28, C45 to C29, C2 to C3, C46 to C30, C47 to C31, C56 to C32, C57 to C33, C58 to C34, C59 to C35, C60 to C36, C61 to C37, C62 to C38, C63 to C39, C3 to C4, C72 to C40, C73 to C41, C74 to C42, C75 to C43, C76 to C44, C77 to C45, C78 to C46, C79 to C47, C80 to C48, C89 to C49, C4 to C5, C90 to C50, C91 to C51, C92 to C52, C93 to C53, C99 to C54, C100 to C55, C101 to C56, C102 to C57, C103 to C58, C108 to C59, C5 to C6, C109 to C60, C112 to C62, C6 to C7, C7 to C8, C8 to C9, D2 to D10, D3 to D11, D4 to D20, D5 to D21, D6 to D51, D7 to D52, D10 to D59, D11 to D60, D12 to D61, L8 to L10, L9 to L11, L2 to L4, L3 to L5, L4 to L6, L5 to L7, L6 to L8, L7 to L9, R116 to R107, R117 to R108, R118 to R109, R119 to R110, R120 to R111, R121 to R112, R122 to R113, R123 to R114, R124 to R115, R141 to R132, R142 to R133, R143 to R134, R144 to R135, R145 to R136, R156 to R147, R157 to R148, R158 to R149, R159 to R150, R160 to R151, R169 to R160, R175 to R165, R178 to R166, R182 to R168, R186 to R171, R39 to R35, R60 to R53, R61 to R54, R62 to R55, R63 to R56, R64 to R57, R65 to R58, R66 to R59, R67 to R60, R68 to R61, R70 to R62, R88 to R79, R89 to R80, R90 to R81, R91 to R82, R92 to R83, R93 to R84, R94 to R85, R95 to R86, R96 to R87, R97 to R88, R98 to R89, R99 to R90, U2 to U1, U1 to U2
Connections:
- net +3V3: now also J13.5 (Pin_5), R10.2, R100.2, R101.2, R102.2, R103.2, R104.2, R105.2, R106.2, R11.2, R12.2, R125.2, R126.2, R127.2, R128.2, R129.2, R13.2, R130.2, R131.2, R137.2, R138.2, R139.2, R14.2, R140.2, R146.2, R15.2, R152.2, R153.2, R154.2, R155.2, R16.2, R17.2, R18.2, R19.2, R20.2, R21.2, R22.2, R23.2, R24.2, R25.2, R36.2, R37.2, R38.2, R40.2, R41.2, R42.2, R43.2, R44.2, R45.2, R46.2, R47.2, R48.2, R49.2, R50.2, R51.2, R69.2, R71.2, R72.2, R73.2, R74.2, R75.2, R76.2, R77.2, R78.2, D57.2 (A), D58.2 (A), R116.2, R117.2, R118.2, R119.2, R120.2, R121.2, R122.2, R123.2, R124.2, R141.2, R142.2, R143.2, R144.2, R145.2, R156.2, R157.2, R158.2, R159.2, R39.2, R63.2, R64.2, R65.2, R66.2, R67.2, R68.2, R70.2, R91.2, R92.2, R93.2, R94.2, R95.2, R96.2, R97.2, R98.2, R99.2, U58.8 (VCC); no longer D8.2 (A), D9.2 (A)
- net +5V: now also R167.2, AD1.2 (B), AD2.2 (B), C61.1, R169.2, U59.1 (VCC)
- net 1-Wire: now also R170.2, U59.2 (IO), WIRE1.1 (A)
- net 1-Wire_OUT: now also R169.1, R170.1
- net Earth: now also C1.2, C10.2, C11.2, D10.2 (A), D11.1 (K), R9.2, SW2.8, U1.5 (GND), U1.6 (GND), U1.7 (GND), U1.8 (GND), U2.1 (-Vin), L2.1, L3.1; no longer R38.2, R48.2, R69.2, R71.2, SW2.4
- net GND: now also C62.1, J1.8 (Pin_8), J13.6 (Pin_6), R163.2, R164.2, U10.3, U11.3, U12.3, U13.3, U14.3, U15.3, U16.3, U17.3, U18.3, U20.3, U21.3, U22.3, U23.3, U24.3, U25.3, U26.3, U27.3, U29.3, U3.3, U30.3, U31.3, U32.3, U33.3, U34.3, U35.3, U36.3, U38.3, U39.3, U4.3, U40.3, U41.3, U42.3, U43.3, U44.3, U45.3, U46.3, U47.3, U48.3, U49.3, U5.3, U50.3, U51.3, U52.3, U53.3, U54.3, U6.3, U60.1 (A1), U60.2 (A0), U60.6 (GND), U7.3, U8.3, U9.3, C61.2, L2.2, L3.2, U58.4 (GND), U59.3 (GND); no longer R36.1, R37.1, R38.1, R48.1
- net GND1: now also SW2.7; no longer SW2.3
- net GND_AA: now also SW2.1, SW2.2; no longer SW2.5, SW2.6
- net I2C_SCL_OUT: now also U58.7 (LY)
- net I2C_SDA_OUT: now also U58.6 (SY)
- net P8.07: now also U39.4, D40.1 (K), R117.1
- net P8.08: now also U38.4, D39.1 (K), R116.1
- net P8.09: now also U36.4, D37.1 (K), R98.1
- net P8.10: now also U35.4, D36.1 (K), R97.1
- net P8.11: now also U34.4, D35.1 (K), R96.1
- net P8.12: now also U33.4, D34.1 (K), R95.1
- net P8.13: now also U32.4, D33.1 (K), R94.1
- net P8.14: now also U31.4, D32.1 (K), R93.1
- net P8.15: now also U30.4, D31.1 (K), R92.1
- net P8.16: now also U29.4, D30.1 (K), R91.1
- net P8.17: now also U22.4, D23.1 (K), R65.1
- net P8.18: now also U21.4, D22.1 (K), R64.1
- net P8.19: now also U20.4, D29.1 (K), R63.1
- net P8.26: now also U27.4, D28.1 (K), R70.1
- net P8.27: now also R69.1, U26.4, D27.1 (K)
- net P8.28: now also U25.4, D26.1 (K), R68.1
- net P8.29: now also U24.4, D25.1 (K), R67.1
- net P8.30: now also U23.4, D24.1 (K), R66.1
- net P8.31: now also R43.1, U18.4, D19.1 (K)
- net P8.32: now also R42.1, U17.4, D18.1 (K)
- net P8.33: now also R41.1, U16.4, D17.1 (K)
- net P8.34: now also R40.1, U15.4, D16.1 (K)
- net P8.35: now also U14.4, D15.1 (K), R39.1
- net P8.36: now also R38.1, U13.4, D14.1 (K); no longer R51.2
- net P8.37: now also R37.1, U12.4, D13.1 (K); no longer R50.2
- net P8.38: now also R36.1, U11.4, D12.1 (K); no longer R49.2
- net P8.39: now also D9.1 (K), R17.1, U10.4; no longer R25.2
- net P8.40: now also D8.1 (K), R16.1, U9.4; no longer R24.2
- net P8.41: now also R15.1, U8.4, D7.1 (K); no longer R23.2
- net P8.42: now also R14.1, U7.4, D6.1 (K); no longer R22.2
- net P8.43: now also R13.1, U6.4, D5.1 (K); no longer R21.2
- net P8.44: now also R12.1, U5.4, D4.1 (K); no longer R20.2
- net P8.45: now also R11.1, U4.4, D3.1 (K); no longer R19.2
- net P8.46: now also R10.1, U3.4, D2.1 (K); no longer R18.2
- net P9.14: now also U40.4, D41.1 (K), R118.1
- net P9.15: now also U41.4, D42.1 (K), R119.1
- net P9.16: now also U42.4, D43.1 (K), R120.1; no longer R137.2
- net P9.17: now also R137.1, U46.4, D46.1 (K)
- net P9.18: now also R138.1, U47.4, D47.1 (K); no longer R152.2
- net P9.21: now also R139.1, U48.4, D48.1 (K); no longer R153.2
- net P9.22: now also R140.1, U49.4, D49.1 (K); no longer R154.2
- net P9.23: now also U50.4, D50.1 (K), R141.1; no longer R155.2
- net P9.25: now also U43.4, D44.1 (K), R121.1; no longer R138.2
- net P9.27: now also U44.4, D45.1 (K), R122.1; no longer R139.2
- net P9.28: now also U45.4, D38.1 (K), R123.1; no longer R140.2
- net P9.29: now also R152.1, U51.4, D53.1 (K)
- net P9.30: now also R153.1, U52.4, D54.1 (K)
- net P9.31: now also R154.1, U53.4, D55.1 (K); no longer R167.2
- net P9.42: now also R155.1, U54.4, D56.1 (K)
- net SCL: now also J13.7 (Pin_7), U58.2 (LX)
- net SCL_5V: now also U59.4 (SCL)
- net SDA: now also J13.8 (Pin_8), U58.3 (SX)
- net SDA_5V: now also U59.5 (SDA)
- net VDD_AA: now also SW2.3, SW2.4; no longer SW2.7, SW2.8
- net at R44.1: now also D12.2 (A); no longer U15.4
- net at R45.1: now also D13.2 (A); no longer U16.4
- net at R46.1: now also D14.2 (A); no longer U17.4
- net at R47.1: now also D15.2 (A); no longer U18.4
- net at R75.1: now also D26.2 (A); no longer U23.4
- net at R76.1: now also D27.2 (A); no longer U24.4
- net at R77.1: now also D28.2 (A); no longer U25.4
- net at R78.1: now also D29.2 (A); no longer U26.4
- net at R128.1: now also D42.2 (A); no longer U41.4
- net at R102.1: now also D33.2 (A); no longer U31.4
- net at R101.1: now also D32.2 (A); no longer U30.4
- net at R100.1: now also D31.2 (A); no longer U29.4
- net at R73.1: now also D24.2 (A); no longer U21.4
- net at R74.1: now also D25.2 (A); no longer U22.4
- net at R125.1: now also D39.2 (A); no longer U38.4
- net at R106.1: now also D37.2 (A); no longer U35.4
- net at R105.1: now also D36.2 (A); no longer U34.4
- net at R104.1: now also D35.2 (A); no longer U33.4
- net at R72.1: now also D23.2 (A); no longer U20.4
- net at R127.1: now also D41.2 (A); no longer U40.4
- net at R103.1: now also D34.2 (A); no longer U32.4
- net at R146.1: now also D50.2 (A); no longer U46.4
- net at R126.1: now also D40.2 (A); no longer U39.4
- net at R164.1: now also AD2.1 (A), U59.7 (AD1); no longer U54.4
- net at R162.2: now also D58.1 (K); no longer D9.1 (K)
- net at R161.2: now also D57.1 (K); no longer D8.1 (K)
- net at D52.1 (K), L7.1: now also SW2.5; no longer SW2.1
- net at D51.1 (K), L4.1: now also SW2.6; no longer SW2.2
- removed net +3.3VA: J13.5 (Pin_5), R10.2, R100.2, R101.2, R102.2, R103.2, R104.2, R105.2, R106.2, R11.2, R12.2, R125.2, R126.2, R127.2, R128.2, R129.2, R13.2, R130.2, R131.2, R14.2, R146.2, R15.2, R16.2, R163.2, R164.2, R17.2, R40.2, R41.2, R42.2, R43.2, R44.2, R45.2, R46.2, R47.2, R72.2, R73.2, R74.2, R75.2, R76.2, R77.2, R78.2
- removed net GND3: J13.6 (Pin_6), R36.2, R37.2, U10.3, U11.3, U12.3, U13.3, U14.3, U15.3, U16.3, U17.3, U18.3, U20.3, U21.3, U22.3, U23.3, U24.3, U25.3, U26.3, U27.3, U29.3, U3.3, U30.3, U31.3, U32.3, U33.3, U34.3, U35.3, U36.3, U38.3, U39.3, U4.3, U40.3, U41.3, U42.3, U43.3, U44.3, U45.3, U46.3, U47.3, U48.3, U49.3, U5.3, U50.3, U51.3, U52.3, U53.3, U54.3, U6.3, U7.3, U8.3, U9.3
- removed net GNDPWR: C1.2, C10.2, C11.2, C62.1, D10.2 (A), D11.1 (K), R69.1, R71.1, R9.2, U1.5 (GND), U1.6 (GND), U1.7 (GND), U1.8 (GND), U2.1 (-Vin), U60.1 (A1), U60.2 (A0), U60.6 (GND)
- new net: D53.2 (A), R156.1
- new net: D6.2 (A), R22.1
- new net: D16.2 (A), R48.1
- new net: Q1.1 (G), U59.6 (PCTLZ)
- new net: Q1.2 (S), WIRE1.2 (B)
- new net: Q1.3 (D), R167.1
- new net: D47.2 (A), R143.1
- new net: D43.2 (A), R129.1
- new net: D9.2 (A), R25.1
- new net: AD1.1 (A), R163.1, U59.8 (AD0)
- new net: D2.2 (A), R18.1
- new net: D55.2 (A), R158.1
- new net: D49.2 (A), R145.1
- new net: D19.2 (A), R51.1
- new net: D18.2 (A), R50.1
- new net: D48.2 (A), R144.1
- new net: D56.2 (A), R159.1
- new net: D4.2 (A), R20.1
- new net: D44.2 (A), R130.1
- new net: D17.2 (A), R49.1
- new net: D22.2 (A), R71.1
- new net: D3.2 (A), R19.1
- new net: D7.2 (A), R23.1
- new net: D45.2 (A), R131.1
- new net: D38.2 (A), R124.1
- new net: D46.2 (A), R142.1
- new net: D5.2 (A), R21.1
- new net: D30.2 (A), R99.1
- new net: D8.2 (A), R24.1
- new net: D54.2 (A), R157.1
- no-connect marks 16 -> 15
Other:
- moved on the sheet: C1, C10, C11, C59, D1, D10, D11, D61, F1, J1, L1, R165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
